File: RangeHood.brd (EAGLE design)
At the start: 100 x 80 mm, 33 parts, among them T1 2N3904

Commit message: Add files via upload
Updates from 3/7/2018. 
Added ground plane; all traces routed.
Parts:
- removed JP6: (no value), pinhead:2X20
- added D2: 1N4004, adafruit:DO41-10
- added FAN1: (no value), pinhead:1X02
- added RL10: 150, adafruit:M0805
- added T2: 2N3904, transistor:TO92
- JP2, JP3, JP4, JP5: device pinhead:2X20 -> pinhead:2X16
- moved JP2 9.67 mm to (31.8, 27.9)
- moved JP3 8.52 mm to (31.8, 22.9)
- moved JP4 7.41 mm to (31.8, 17.8)
- moved JP5 6.35 mm to (31.8, 12.7)
- moved BUZZER 5.08 mm to (3.81, 72.4)
- moved D1 3.81 mm to (8.89, 71.1)
- moved JP1 1.31 mm to (43.8, 44.6)
- moved LED1 1.27 mm to (26.7, 67.3)
- moved LED2 1.27 mm to (36.8, 67.3)
- moved LED3 1.27 mm to (48.3, 67.3)
- moved RL1 1.27 mm to (82.5, 64.8)
- moved RL3 1.27 mm to (80.0, 64.8)
- moved RL5 1.27 mm to (77.5, 64.8)
- moved RL7 1.27 mm to (74.9, 64.8)
Connections:
- new net N$12: RL10.1, T2.2
- new net N$6: D2.A, FAN1.2, T2.1
- net +3V3: now also JP1.1, JP1.17, JP2.10, JP2.12, JP2.14, JP2.16, JP2.18, JP2.2, JP2.20, JP2.22, JP2.24, JP2.26, JP2.28, JP2.30, JP2.32, JP2.4, JP2.6, JP2.8
- net +5V: now also D2.C, FAN1.1, JP1.2, JP1.4, JP5.1, JP5.11, JP5.13, JP5.15, JP5.17, JP5.19, JP5.21, JP5.23, JP5.25, JP5.27, JP5.29, JP5.3, JP5.31, JP5.5, JP5.7, JP5.9
- net GND: now also JP1.14, JP1.20, JP1.25, JP1.30, JP1.34, JP1.39, JP1.6, JP1.9, JP5.10, JP5.12, JP5.14, JP5.16, JP5.18, JP5.2, JP5.20, JP5.22, JP5.24, JP5.26, JP5.28, JP5.30, JP5.32, JP5.4, JP5.6, JP5.8, T2.3
- net GPIO10: now also JP1.19
- net GPIO11: now also JP1.23
- net GPIO12: now also JP1.32
- net GPIO13: now also JP1.33, RL10.2
- net GPIO14: now also JP1.8
- net GPIO15: now also JP1.10
- net GPIO16: now also JP1.36
- net GPIO17: now also JP1.11
- net GPIO18: now also JP1.12
- net GPIO19: now also JP1.35
- net GPIO20: now also JP1.38
- net GPIO21: now also JP1.40
- net GPIO22: now also JP1.15
- net GPIO23: now also JP1.16
- net GPIO24: now also JP1.18
- net GPIO25: now also JP1.22
- net GPIO26: now also JP1.37
- net GPIO27: now also JP1.13
- net GPIO4: now also JP1.7
- net GPIO5: now also JP1.29
- net GPIO6: now also JP1.31
- net GPIO7: now also JP1.26
- net GPIO8: now also JP1.24
- net GPIO9: now also JP1.21
- net N$23: now also JP1.27
- net N$31: now also JP1.28
- net SCL: now also JP1.5
- net SDA: now also JP1.3
Routing:
- net GND: track 282.5 -> 49.2 mm, vias 0 -> 1
- net +5V: track 174.2 -> 288.7 mm, vias 0 -> 1
- net GPIO13: track 0.00 -> 57.9 mm, vias 0 -> 1
- net GPIO26: track 21.4 -> 77.6 mm, vias 0 -> 1
- net GPIO5: track 54.3 -> 11.3 mm
- net +3V3: track 170.9 -> 207.2 mm, vias 0 -> 1
- net N$12: track 40.0 -> 4.13 mm, vias 1 -> 0
- net N$6: track 0.00 -> 17.6 mm
- net GPIO6: track 23.7 -> 40.1 mm
- net GPIO19: track 45.4 -> 60.9 mm
- net GPIO18: track 25.5 -> 38.9 mm
- net SCL: track 75.5 -> 87.6 mm, vias 0 -> 1
- net GPIO21: track 25.0 -> 36.8 mm
- net GPIO12: track 0.00 -> 11.3 mm
- net N$31: track 0.00 -> 11.3 mm
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- added copper zone on layer 16, net GND
Other:
- board text added: "3.3v"
- board text added: "5V"
- board text added: "GND"
- board text added: "James O'Gorman Smart Range Hood 2018 Pi Chef Challenge"
- board text added: "Rev 0.1"

Commit message: Add files via upload
Connections:
- net GPIO12: now also Q3.1
- net GPIO20: no longer Q3.1
Routing:
- net GPIO20: track 46.7 -> 11.3 mm
- net GPIO12: track 11.3 -> 41.8 mm
- net N$2: track 49.6 -> 55.3 mm, vias 0 -> 1
- net GND: vias 1 -> 2
Other:
- board text added: "*"
- board text added: "MQ4"
- board text added: "MQ4 - Methane MQ6 - LPG MQ7 - CO MQ8 - Hydrogen"
- board text added: "MQ6"
- board text added: "MQ7"
- board text added: "MQ8"
Changed lines of the file:
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@@
 Pi Chef Challenge</text>
 <text x="79.756" y="6.985" size="1.27" layer="25">Rev 0.1</text>
+<text x="85.344" y="48.133" size="1.27" layer="25">MQ4 - Methane
+MQ6 - LPG
+MQ7 - CO
+MQ8 - Hydrogen</text>
+<text x="62.865" y="70.993" size="1.27" layer="25">MQ8</text>
+<text x="48.895" y="70.993" size="1.27" layer="25">MQ7</text>
+<text x="37.465" y="70.993" size="1.27" layer="25">MQ6</text>
+<text x="26.035" y="70.993" size="1.27" layer="25">MQ4</text>
+<text x="5.08" y="37.211" size="1.27" layer="25">*</text>
+<text x="2.032" y="41.783" size="1.27" layer="25">*</text>
+<text x="4.699" y="74.295" size="1.27" layer="25">*</text>
+<text x="76.708" y="41.91" size="1.27" layer="25">*</text>
+<text x="66.802" y="4.191" size="1.27" layer="25">*</text>
 </plain>
 <attributes>
@@
 </element>
 <element name="LED3" library="adafruit" library_urn="urn:adsk.eagle:library:420" package="LED3MM" value="" x="48.26" y="67.31" smashed="yes" rot="R90">
-<attribute name="NAME" x="54.61" y="68.961" size="1.27" layer="25" ratio="10" rot="R180"/>
+<attribute name="NAME" x="54.61" y="67.691" size="1.27" layer="25" ratio="10" rot="R180"/>
 <attribute name="VALUE" x="49.911" y="69.215" size="1.27" layer="27" ratio="10" rot="R90"/>
 </element>
@@
 <contactref element="JP5" pad="30"/>
 <contactref element="JP5" pad="32"/>
-<polygon width="0.254" layer="16" isolate="0.4064">
-<vertex x="0.381" y="79.502"/>
-<vertex x="99.568" y="79.502"/>
-<vertex x="99.568" y="0.508"/>
-<vertex x="0.381" y="0.508"/>
-</polygon>
 <wire x1="74.93" y1="63.82" x2="82.55" y2="63.82" width="0.8128" layer="1"/>
 <wire x1="82.55" y1="63.82" x2="82.616" y2="63.754" width="0.8128" layer="1" curve="90"/>
@@
 <wire x1="68.961" y1="44.323" x2="67.945" y2="43.307" width="0.2032" layer="1"/>
 <via x="3.81" y="67.31" extent="1-16" drill="1.27" diameter="1.905" shape="square"/>
+<via x="54.61" y="69.342" extent="1-16" drill="0.762" diameter="1.2954"/>
+<polygon width="0.2032" layer="16" isolate="0.4064">
+<vertex x="0.381" y="79.502"/>
+<vertex x="99.568" y="79.502"/>
+<vertex x="99.568" y="0.254"/>
+<vertex x="0.381" y="0.254"/>
+<vertex x="0.381" y="59.182"/>
+<vertex x="0.889" y="59.69"/>
+<vertex x="6.858" y="59.817"/>
+<vertex x="6.858" y="66.167"/>
+<vertex x="1.27" y="66.04"/>
+<vertex x="0.381" y="66.929"/>
+</polygon>
 <wire x1="77.47" y1="63.82" x2="80.01" y2="63.82" width="0" layer="19" extent="1-1"/>
 <wire x1="82.55" y1="63.82" x2="80.01" y2="63.82" width="0" layer="19" extent="1-1"/>
-<wire x1="50.2666" y1="53.7718" x2="55.3466" y2="56.3118" width="0" layer="19" extent="1-1"/>
-<wire x1="29.9466" y1="53.7718" x2="24.8666" y2="56.3118" width="0" layer="19" extent="1-1"/>
 </signal>
 <signal name="GPIO18">
@@
 <wire x1="63.881" y1="46.26784375" x2="63.881" y2="44.323" width="0.2032" layer="1"/>
 <wire x1="63.881" y1="44.323" x2="62.865" y2="43.307" width="0.2032" layer="1"/>
-<wire x1="57.531" y1="60.833" x2="59.436" y2="58.928" width="0.2032" layer="16" curve="90"/>
-<wire x1="59.436" y1="58.928" x2="63.754" y2="58.928" width="0.2032" layer="16"/>
-<wire x1="63.754" y1="58.928" x2="64.262" y2="58.42" width="0.2032" layer="16" curve="-90"/>
-<wire x1="64.262" y1="58.42" x2="64.262" y2="54.864" width="0.2032" layer="16"/>
-<wire x1="57.531" y1="66.548" x2="57.531" y2="66.04" width="0.2032" layer="16"/>
-<wire x1="57.531" y1="66.04" x2="57.531" y2="60.833" width="0.2032" layer="16"/>
-<wire x1="64.262" y1="54.864" x2="62.9666" y2="53.7718" width="0.2032" layer="16"/>
-<wire x1="57.531" y1="66.548" x2="57.531" y2="70.104" width="0.2032" layer="16"/>
+<wire x1="57.531" y1="70.104" x2="57.531" y2="60.96" width="0.2032" layer="16"/>
+<wire x1="57.531" y1="60.96" x2="57.531" y2="60.833" width="0.2032" layer="16"/>
 <wire x1="57.531" y1="70.104" x2="57.023" y2="70.612" width="0.2032" layer="16" curve="90"/>
 <wire x1="34.925" y1="70.612" x2="34.29" y2="71.247" width="0.2032" layer="16" curve="-90"/>
 <wire x1="34.29" y1="71.247" x2="34.29" y2="74.93" width="0.2032" layer="16"/>
 <wire x1="57.023" y1="70.612" x2="34.925" y2="70.612" width="0.2032" layer="16"/>
+<wire x1="57.531" y1="60.833" x2="57.531" y2="58.293" width="0.2032" layer="16"/>
+<wire x1="57.531" y1="58.293" x2="56.515" y2="57.277" width="0.2032" layer="16" curve="90"/>
+<wire x1="56.515" y1="57.277" x2="56.515" y2="55.753" width="0.2032" layer="16"/>
+<wire x1="56.515" y1="55.753" x2="57.277" y2="54.991" width="0.2032" layer="16" curve="90"/>
+<wire x1="57.277" y1="54.991" x2="61.976" y2="54.991" width="0.2032" layer="16"/>
+<wire x1="61.976" y1="54.991" x2="62.9666" y2="54.0004" width="0.2032" layer="16" curve="-90"/>
+<wire x1="62.9666" y1="54.0004" x2="62.9666" y2="53.7718" width="0.2032" layer="16"/>
 </signal>
 <signal name="GPIO21">
@@
 <signal name="GPIO20">
 <contactref element="PCB1" pad="P$38"/>
-<contactref element="Q3" pad="1"/>
 <contactref element="JP1" pad="38"/>
-<wire x1="65.405" y1="52.43655625" x2="65.405" y2="45.847" width="0.2032" layer="1"/>
-<wire x1="64.4906" y1="53.35095625" x2="65.405" y2="52.43655625" width="0.2032" layer="1"/>
+<wire x1="64.4906" y1="53.35095625" x2="64.77" y2="53.07155625" width="0.2032" layer="1"/>
 <wire x1="65.5066" y1="56.3118" x2="64.4906" y2="55.2958" width="0.2032" layer="1"/>
 <wire x1="64.4906" y1="55.2958" x2="64.4906" y2="53.35095625" width="0.2032" layer="1"/>
-<wire x1="58.039" y1="60.833" x2="59.563" y2="59.309" width="0.2032" layer="16" curve="90"/>
-<wire x1="64.135" y1="59.309" x2="65.5066" y2="57.9374" width="0.2032" layer="16" curve="-90"/>
-<wire x1="65.5066" y1="57.9374" x2="65.5066" y2="56.3118" width="0.2032" layer="16"/>
-<wire x1="59.563" y1="59.309" x2="64.135" y2="59.309" width="0.2032" layer="16"/>
-<wire x1="45.72" y1="74.93" x2="45.72" y2="72.39" width="0.2032" layer="16"/>
-<wire x1="45.72" y1="72.39" x2="46.99" y2="71.12" width="0.2032" layer="16" curve="90"/>
-<wire x1="46.99" y1="71.12" x2="57.15" y2="71.12" width="0.2032" layer="16"/>
-<wire x1="57.15" y1="71.12" x2="58.039" y2="70.231" width="0.2032" layer="16" curve="-90"/>
-<wire x1="58.039" y1="70.231" x2="58.039" y2="60.833" width="0.2032" layer="16"/>
+<wire x1="64.77" y1="46.482" x2="65.405" y2="45.847" width="0.2032" layer="1"/>
+<wire x1="64.77" y1="53.07155625" x2="64.77" y2="46.482" width="0.2032" layer="1"/>
 </signal>
 <signal name="GPIO16">
@@
 <wire x1="58.9026" y1="54.19264375" x2="57.8866" y2="55.20864375" width="0.2032" layer="1"/>
 <wire x1="57.8866" y1="55.20864375" x2="57.8866" y2="56.3118" width="0.2032" layer="1"/>
+<contactref element="Q3" pad="1"/>
+<wire x1="45.72" y1="74.93" x2="45.72" y2="71.12" width="0.2032" layer="16"/>
+<wire x1="45.72" y1="71.12" x2="57.023" y2="71.12" width="0.2032" layer="16"/>
+<wire x1="57.023" y1="71.12" x2="58.039" y2="70.104" width="0.2032" layer="16" curve="-90"/>
+<wire x1="58.039" y1="58.039" x2="57.8866" y2="57.8866" width="0.2032" layer="16" curve="90"/>
+<wire x1="57.8866" y1="57.8866" x2="57.8866" y2="56.3118" width="0.2032" layer="16"/>
+<wire x1="58.039" y1="70.104" x2="58.039" y2="58.039" width="0.2032" layer="16"/>
 </signal>
 <signal name="N$31">
@@
 <contactref element="LED3" pad="K"/>
 <wire x1="48.26" y1="74.93" x2="51.1556" y2="77.8256" width="0.3048" layer="1"/>
-<wire x1="51.1556" y1="77.8256" x2="87.2744" y2="77.8256" width="0.3048" layer="1"/>
+<wire x1="51.1556" y1="77.8256" x2="54.61" y2="77.8256" width="0.3048" layer="1"/>
+<wire x1="54.61" y1="77.8256" x2="87.2744" y2="77.8256" width="0.3048" layer="1"/>
 <wire x1="87.63" y1="74.93" x2="87.63" y2="77.47" width="0.3048" layer="1"/>
 <wire x1="87.63" y1="77.47" x2="87.2744" y2="77.8256" width="0.3048" layer="1"/>
 <wire x1="48.26" y1="74.93" x2="48.26" y2="68.58" width="0.2032" layer="1"/>
+<via x="54.61" y="72.136" extent="1-16" drill="0.762" diameter="1.3"/>
+<wire x1="54.61" y1="77.8256" x2="54.61" y2="72.136" width="0.3048" layer="1"/>
 </signal>
 <signal name="N$6">
