File: RangeHood.sch (EAGLE design)
At the start: 33 parts, among them T1 2N3904

Commit message: Add files via upload
Updates from 3/7/2018. 
Added ground plane; all traces routed.
Parts:
- removed JP6: (no value), pinhead:PINHD-2X20
- added D2: 1N4004, adafruit:1N4004
- added FAN1: (no value), pinhead:PINHD-1X2
- added RL10: 150, adafruit:R-US_M0805
- added T2: 2N3904, transistor:2N3904
- JP2, JP3, JP4, JP5: device pinhead:PINHD-2X20 -> pinhead:PINHD-2X16
Connections:
- new net N$12: RL10.1, T2.B
- new net N$6: D2.A, FAN1.2, T2.C
- net +3V3: now also JP1.1, JP1.17, JP2.10, JP2.12, JP2.14, JP2.16, JP2.18, JP2.2, JP2.20, JP2.22, JP2.24, JP2.26, JP2.28, JP2.30, JP2.32, JP2.4, JP2.6, JP2.8
- net +5V: now also D2.C, FAN1.1, JP1.2, JP1.4, JP5.1, JP5.11, JP5.13, JP5.15, JP5.17, JP5.19, JP5.21, JP5.23, JP5.25, JP5.27, JP5.29, JP5.3, JP5.31, JP5.5, JP5.7, JP5.9
- net GND: now also JP1.14, JP1.20, JP1.25, JP1.30, JP1.34, JP1.39, JP1.6, JP1.9, JP5.10, JP5.12, JP5.14, JP5.16, JP5.18, JP5.2, JP5.20, JP5.22, JP5.24, JP5.26, JP5.28, JP5.30, JP5.32, JP5.4, JP5.6, JP5.8, T2.E
- net GPIO10: now also JP1.19
- net GPIO11: now also JP1.23
- net GPIO12: now also JP1.32
- net GPIO13: now also JP1.33, RL10.2
- net GPIO14: now also JP1.8
- net GPIO15: now also JP1.10
- net GPIO16: now also JP1.36
- net GPIO17: now also JP1.11
- net GPIO18: now also JP1.12
- net GPIO19: now also JP1.35
- net GPIO20: now also JP1.38
- net GPIO21: now also JP1.40
- net GPIO22: now also JP1.15
- net GPIO23: now also JP1.16
- net GPIO24: now also JP1.18
- net GPIO25: now also JP1.22
- net GPIO26: now also JP1.37
- net GPIO27: now also JP1.13
- net GPIO4: now also JP1.7
- net GPIO5: now also JP1.29
- net GPIO6: now also JP1.31
- net GPIO7: now also JP1.26
- net GPIO8: now also JP1.24
- net GPIO9: now also JP1.21
- net N$23: now also JP1.27
- net N$31: now also JP1.28
- net SCL: now also JP1.5
- net SDA: now also JP1.3
Other:
- moved on the sheet: JP1

Commit message: Add files via upload
Connections:
- net GPIO12: now also Q3.G
- net GPIO20: no longer Q3.G
Other:
- note added: "MQ4 - Methane"
- note added: "MQ6 - LPG"
- note added: "MQ7 - CO"
- note added: "MQ8 - Hydrogen"
Changed lines of the file:
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@@
 GPIO24 - Med
 GPIO23 - Low</text>
+<text x="83.82" y="114.3" size="1.778" layer="91">MQ4 - Methane</text>
+<text x="81.28" y="68.58" size="1.778" layer="91">MQ6 - LPG</text>
+<text x="83.82" y="20.32" size="1.778" layer="91">MQ7 - CO</text>
+<text x="83.82" y="-22.86" size="1.778" layer="91">MQ8 - Hydrogen</text>
 </plain>
 <instances>
@@
 </segment>
 <segment>
+<pinref part="JP1" gate="A" pin="38"/>
+<wire x1="-96.52" y1="185.42" x2="-96.52" y2="195.58" width="0.1524" layer="91"/>
+<label x="-96.52" y="193.04" size="1.778" layer="95" rot="R90"/>
+</segment>
+</net>
+<net name="GPIO16" class="0">
+<segment>
+<pinref part="PCB1" gate="G$1" pin="GPIO16"/>
+<wire x1="-73.66" y1="147.32" x2="-73.66" y2="160.02" width="0.1524" layer="91"/>
+<label x="-73.66" y="154.94" size="1.778" layer="95" rot="R90"/>
+</segment>
+<segment>
+<pinref part="JP1" gate="A" pin="36"/>
+<wire x1="-99.06" y1="185.42" x2="-99.06" y2="195.58" width="0.1524" layer="91"/>
+<label x="-99.06" y="193.04" size="1.778" layer="95" rot="R90"/>
+</segment>
+</net>
+<net name="GPIO12" class="0">
+<segment>
+<pinref part="PCB1" gate="G$1" pin="GPIO12"/>
+<wire x1="-83.82" y1="147.32" x2="-83.82" y2="160.02" width="0.1524" layer="91"/>
+<label x="-83.82" y="154.94" size="1.778" layer="95" rot="R90"/>
+</segment>
+<segment>
+<pinref part="JP1" gate="A" pin="32"/>
+<wire x1="-104.14" y1="185.42" x2="-104.14" y2="195.58" width="0.1524" layer="91"/>
+<label x="-104.14" y="193.04" size="1.778" layer="95" rot="R90"/>
+</segment>
+<segment>
 <pinref part="Q3" gate="G$1" pin="G"/>
 <wire x1="109.22" y1="-2.54" x2="96.52" y2="-2.54" width="0.1524" layer="91"/>
 <label x="96.52" y="-2.54" size="1.778" layer="95"/>
 </segment>
-<segment>
-<pinref part="JP1" gate="A" pin="38"/>
-<wire x1="-96.52" y1="185.42" x2="-96.52" y2="195.58" width="0.1524" layer="91"/>
-<label x="-96.52" y="193.04" size="1.778" layer="95" rot="R90"/>
-</segment>
-</net>
-<net name="GPIO16" class="0">
-<segment>
-<pinref part="PCB1" gate="G$1" pin="GPIO16"/>
-<wire x1="-73.66" y1="147.32" x2="-73.66" y2="160.02" width="0.1524" layer="91"/>
-<label x="-73.66" y="154.94" size="1.778" layer="95" rot="R90"/>
-</segment>
-<segment>
-<pinref part="JP1" gate="A" pin="36"/>
-<wire x1="-99.06" y1="185.42" x2="-99.06" y2="195.58" width="0.1524" layer="91"/>
-<label x="-99.06" y="193.04" size="1.778" layer="95" rot="R90"/>
-</segment>
-</net>
-<net name="GPIO12" class="0">
-<segment>
-<pinref part="PCB1" gate="G$1" pin="GPIO12"/>
-<wire x1="-83.82" y1="147.32" x2="-83.82" y2="160.02" width="0.1524" layer="91"/>
-<label x="-83.82" y="154.94" size="1.778" layer="95" rot="R90"/>
-</segment>
-<segment>
-<pinref part="JP1" gate="A" pin="32"/>
-<wire x1="-104.14" y1="185.42" x2="-104.14" y2="195.58" width="0.1524" layer="91"/>
-<label x="-104.14" y="193.04" size="1.778" layer="95" rot="R90"/>
-</segment>
-</net>
+</net>
